Commit message: Update robot.urdf

File: urdf/robot.urdf (robot description, URDF)
Before this commit: robot myrobot, 9 links, 8 joints
Links:
- link link0: geometry collision cylinder length=3 radius=0.35; visual cylinder length=3 radius=0.35
- link link2: geometry collision cylinder length=2 radius=0.1; visual cylinder length=2 radius=0.1
Joints:
- joint link0_to_link1: origin xyz=0 0 2 rpy=0 0 0 -> xyz=0 0 3 rpy=0 0 0
- joint sphere2_to_link2: origin xyz=0 0 3.5 rpy=0 0 0 -> xyz=0 0 2 rpy=0 0 0

Commit message: Update robot.urdf

File: urdf/robot.urdf (robot description, URDF)
Before this commit: robot myrobot, 9 links, 8 joints
Links:
- link link0: geometry collision cylinder length=4 radius=0.35; visual cylinder length=4 radius=0.35
- link link1: geometry collision cylinder length=3.2 radius=0.2; visual cylinder length=3.2 radius=0.2
- link link2: geometry collision cylinder length=2.8 radius=0.1; visual cylinder length=2.8 radius=0.1
Joints:
- joint link0_to_link1: origin xyz=0 0 3 rpy=0 0 0 -> xyz=0 0 4 rpy=0 0 0
- joint link1_to_link2: origin xyz=0 0 3 rpy=0 0 0 -> xyz=0 0 3.2 rpy=0 0 0
- joint sphere2_to_link2: origin xyz=0 0 2 rpy=0 0 0 -> xyz=0 0 2.8 rpy=0 0 0
